File: headstage-64.sch (EAGLE design)
At the start: 195 parts, among them J8 DF40C-70DP-0.4V(51), J9 PINHD-1X5_HALF_CONNETOR, U1 ADA4062-4ACPZ-R7, U10 BNO055, U11 TS4231, U12 TS4231, U13 TLV70733, U14 10M08DC, U15 TLV70733, U16 LT3463, U17 TLV70725, U18 TPS62621, U19 ASCO-50.000MHZ-EK-T3, U2 AD5681RBCPZ-1RL7, U20 TLV70712, U3 CAT4016_QFN, U4 TPL0501_UQFN, U5 DG509B, U6 TS4231, U7 RHD2064_BGA, U8 TS4231, U9 DS90UB913A_WQFN

Commit message: onix-headstage-64 rev. 1.3B
- This is a patch ("B") on rev. 1.3, the beta-test version, that addresses
difficulties with assembly and use
- Assembly differences:
    - R45 has been adjusted right by 0.2 mm
    - C75-77 have been added to address noise leaking from vcoax into
    electrodes.
    - The adapter boards have been removed from the design. This results
    in non-contiguous reference designators, but components names have
    NOT been changed
- Copper pours have been added to all layers to aid with ease of pcb fab
and improve thermal performance
- Thermal reliefs have been added to contacts onto copper pours except
those where head dissipation is critical (power supplies)
Parts:
- removed D1, D2, D3: SESD0402X1UN-0020-090, jonnew:Z-DIODE_0402T-DFN
- removed J1, J3, J6: (no value), jonnew:COAX_XFL
- removed J2, J4, J7: (no value), jonnew:PINHD-1X4HEADSTAGE64-DAUGHTER-CARD-CASTELLATED
- removed L1, L3, L5: CIG21L4R7MNE, jonnew:L_0805T
- removed R20, R3, R9: 1k, jonnew:R_0201T
- added C74, C75, C77: 10uF, jonnew:C_0402T
- J9: value PINHD-1X5_HALF_CONNETOR -> (none); device jonnew:PINHD-1X5_HALF_CONNETOR -> jonnew:PINHD-1X5_HALF_CONNECTOR
- U9: value DS90UB913A_WQFN -> (none)
Connections:
- removed net GND1: D2.A, J3.2, J4.2, J4.4
- removed net GND2: D1.A, J1.2, J2.2, J2.4
- removed net GND3: D3.A, J6.2, J7.2, J7.4
- removed net N$25: J4.1, L3.2, R9.2
- removed net N$48: J2.1, L1.2, R3.2
- removed net N$50: J7.1, L5.2, R20.2
- removed net _SIGOUT: D2.C, J3.1, J4.3, L3.1, R9.1
- removed net _SIGOUT1: D1.C, J1.1, J2.3, L1.1, R3.1
- removed net _SIGOUT2: D3.C, J6.1, J7.3, L5.1, R20.1
- net ESTIM_POW_EN: now also U14G$6.DIFFIO_RX_T18P/DEV_OE/A6; no longer U14G$6.DIFFIO_RX_T18P/DEV_OEA6
- net GND: now also C74.2, C75.2, C77.2
- net VCOAX: now also C74.1, C75.1, C77.1
Other:
- note added: "ADAPTER INPUT"
- note removed: "INPUT"
- note removed: "NB: IO daughter boards. Multiple allows them to be replaced if coax connector gets worn out."
- moved on the sheet: C6, C7, J5, J9, L2, L4, R10
