File: headstage-64.brd (EAGLE design)
At the start: 19 x 19 mm, 183 parts, among them J8 DF40C-70DP-0.4V(51), U1 ADA4062-4ACPZ-R7, U10 BNO055, U11 TS4231, U12 TS4231, U13 TLV70733, U14 10M08DC, U15 TLV70733, U16 LT3463, U17 TLV70725, U18 TPS62621, U19 ASCO-50.000MHZ-EK-T3, U2 AD5681RBCPZ-1RL7, U20 TLV70712, U3 CAT4016_QFN, U4 TPL0501_UQFN, U5 DG509B, U6 TS4231, U7 RHD2064_BGA, U8 TS4231

Commit message: Replace every bulk cap on Vcoax with 10uF
- To reduce near DC noise coming from power over coax and reduce BOM complexity
Parts:
- C37, C39, C41, C55: value 1uF -> 10uF
- C69: value 2.2uF -> 10uF
Changed lines of the file:
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@@
 <element name="R46" library="jonnew" package="0201T" value="90.9k" x="-8.13" y="2.64" smashed="yes"/>
 <element name="C57" library="jonnew" package="0201T" value="10pF" x="-6.6" y="6.33" smashed="yes" rot="R45"/>
-<element name="C39" library="jonnew" package="0402T" value="1uF" x="0.44" y="2.16" smashed="yes" rot="R90">
+<element name="C39" library="jonnew" package="0402T" value="10uF" x="0.44" y="2.16" smashed="yes" rot="R90">
 <attribute name="PARTNO" value="CL05A105KO5NNNC" x="0.44" y="2.16" size="1.778" layer="27" rot="R90" display="off"/>
 </element>
@@
 <attribute name="PARTNO" value="CL05A105KO5NNNC" x="6.96" y="2.38" size="1.778" layer="27" rot="R90" display="off"/>
 </element>
-<element name="C55" library="jonnew" package="0402T" value="1uF" x="2.42" y="2.22" smashed="yes" rot="R90">
+<element name="C55" library="jonnew" package="0402T" value="10uF" x="2.42" y="2.22" smashed="yes" rot="R90">
 <attribute name="PARTNO" value="CL05A105KO5NNNC" x="2.42" y="2.22" size="1.778" layer="27" rot="R90" display="off"/>
 </element>
-<element name="C41" library="jonnew" package="0402T" value="1uF" x="-1.34" y="3.23" smashed="yes">
+<element name="C41" library="jonnew" package="0402T" value="10uF" x="-1.34" y="3.23" smashed="yes">
 <attribute name="PARTNO" value="CL05A105KO5NNNC" x="-1.34" y="3.23" size="1.778" layer="27" display="off"/>
 </element>
@@
 <element name="C30" library="jonnew" package="0201T" value="0.1uF" x="-5.21" y="-6.35" smashed="yes" rot="MR180"/>
 <element name="U13" library="jonnew" package="X2SON" value="TLV70733" x="-7.7084375" y="-2.3689875" smashed="yes" rot="MR60.9"/>
-<element name="C37" library="jonnew" package="0402T" value="1uF" x="-8.37941875" y="-1.369096875" smashed="yes" rot="MR330.9">
+<element name="C37" library="jonnew" package="0402T" value="10uF" x="-8.37941875" y="-1.369096875" smashed="yes" rot="MR330.9">
 <attribute name="PARTNO" value="CL05A105KO5NNNC" x="-9.4106125" y="0.6892125" size="1.778" layer="28" rot="MR330.9" display="off"/>
 </element>
@@
 <element name="R44" library="jonnew" package="0201T" value="4.7k" x="7.8" y="-4.3" smashed="yes" rot="R180"/>
 <element name="U18" library="jonnew" package="XBGA6_1.2X0.8" value="TPS62621" x="4.92" y="2.34" smashed="yes" rot="R270"/>
-<element name="C69" library="jonnew" package="0402T" value="2.2uF" x="4.74" y="3.26" smashed="yes">
+<element name="C69" library="jonnew" package="0402T" value="10uF" x="4.74" y="3.26" smashed="yes">
 <attribute name="PARTNO" value="CL05A105KO5NNNC" x="4.74" y="8.14" size="1.778" layer="27" display="off"/>
 </element>

Commit message: 22uF caps replaced with 15uF due to ease of sourcing.
Parts:
- C24, C73: value 22uF -> 15uF
Changed lines of the file:
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@@
 </element>
 <element name="R25" library="jonnew" package="0201T" value="49.9" x="3.05" y="-0.15" smashed="yes"/>
-<element name="C24" library="jonnew" package="0402T" value="22uF" x="-0.61" y="-1.12" smashed="yes" rot="R180">
+<element name="C24" library="jonnew" package="0402T" value="15uF" x="-0.61" y="-1.12" smashed="yes" rot="R180">
 <attribute name="PARTNO" value="CL05A226MQ5QUNC" x="-0.61" y="-1.12" size="1.778" layer="27" rot="R180" display="off"/>
 </element>
@@
 <attribute name="PARTNO" value="CL03A105MP3ZSNH" x="-0.2658" y="6.2596" size="1.778" layer="28" rot="MR0" display="off"/>
 </element>
-<element name="C73" library="jonnew" package="0402T" value="22uF" x="7.26" y="3.53" smashed="yes" rot="R180">
+<element name="C73" library="jonnew" package="0402T" value="15uF" x="7.26" y="3.53" smashed="yes" rot="R180">
 <attribute name="PARTNO" value="CL05A226MQ6ZUN8" x="7.26" y="3.53" size="1.778" layer="27" rot="R180" display="off"/>
 </element>
